File: Gmouse/Gmouse.kicad_sch (KiCad schematic)
At the start: 84 parts, among them J1 Motor_RF, J2 Motor_RR, J3 Motor_LF, J4 Motor_LR, J5 Conn_01x08_Pin, Q1 NMOS, Q10 SFH300, Q11 NMOS, Q12 SFH300, Q14 BC847, Q2 SFH300, Q3 NMOS, Q4 SFH300, Q5 NMOS, Q6 SFH300, Q7 NMOS, Q8 SFH300, Q9 NMOS, SW1 SW_SPDT, U1 Teensy4.0, U2 TB6612FNG, U4 HCMS-2903, U5 TB6612FNG, U6 LD1117S50TR_SOT223, U7 LD1117S33TR_SOT223

Commit message: cleaned up IR Emitter Circuit
Parts:
- added C21, C23: 4.7uF, Capacitor_SMD:C_1206_3216Metric_Pad1.33x1.80mm_HandSolder, symbol Device:C_Small
- added C22, C24: 0.1uF, Capacitor_SMD:C_1206_3216Metric_Pad1.33x1.80mm_HandSolder, symbol Device:C_Small
- added D10, D11, D12, D13, D8, D9: IR, LED_THT:LED_D5.0mm_Horizontal_O3.81mm_Z9.0mm, symbol Device:LED
- added Q13, Q15: NMOS, Package_TO_SOT_SMD:SOT-23, symbol Simulation_SPICE:NMOS
- added R28: 10K, Resistor_SMD:R_1206_3216Metric_Pad1.30x1.75mm_HandSolder, symbol Device:R
- added R29, R32: 100, Resistor_SMD:R_1206_3216Metric_Pad1.30x1.75mm_HandSolder, symbol Device:R
- added R30, R33: 47K, Resistor_SMD:R_1206_3216Metric_Pad1.30x1.75mm_HandSolder, symbol Device:R
- added R31, R34: 51, Resistor_SMD:R_1206_3216Metric_Pad1.30x1.75mm_HandSolder, symbol Device:R
- C1, C10, C3, C8: footprint (none) -> Capacitor_SMD:CP_Elec_4x5.4
- D7: footprint (none) -> Diode_SMD:D_SOD-323_HandSoldering
- Q1, Q11, Q3, Q5, Q7, Q9: footprint (none) -> Package_TO_SOT_SMD:SOT-23
Connections:
- net +3V3: now also U4.10 (SEL), U4.11 (V_LOGIC), C21.1, C22.1, C23.1, C24.1, R28.2, R31.1, R34.1
- net +5V: no longer U4.10 (SEL), U4.11 (V_LOGIC)
- net GND: now also Q1.2 (S), Q11.2 (S), Q3.2 (S), Q5.2 (S), Q7.2 (S), Q9.2 (S), C21.2, C22.2, C23.2, C24.2, Q13.2 (S), Q15.2 (S), R30.2, R33.2; no longer Q1.3 (S), Q11.3 (S), Q3.3 (S), Q5.3 (S), Q7.3 (S), Q9.3 (S)
- net HCMS_CE: now also U1.12 (10_CS_MQSR)
- net HCMS_RS: now also U1.14 (12_MISO_MQSL)
- net IR_Emmiter_Left_Half: now also R29.1
- net IR_Emmiter_Right_Half: now also R32.1
- net Interface_Button1: now also U1.45 (34_DAT1_MISO2)
- net Interface_Button2: now also U1.46 (35_DAT0_MOSI2)
- net at R21.2, R22.1: now also Q11.1 (G); no longer Q11.2 (G)
- net at R13.2, R14.1: now also Q7.1 (G); no longer Q7.2 (G)
- net at R5.2, R6.1: now also Q3.1 (G); no longer Q3.2 (G)
- net at D5.1 (K): now also Q9.3 (D); no longer Q9.1 (D)
- net at R10.1, R9.2: now also Q5.1 (G); no longer Q5.2 (G)
- net at D4.1 (K): now also Q7.3 (D); no longer Q7.1 (D)
- net at D6.1 (K): now also Q11.3 (D); no longer Q11.1 (D)
- net at D2.1 (K): now also Q3.3 (D); no longer Q3.1 (D)
- net at R17.2, R18.1: now also Q9.1 (G); no longer Q9.2 (G)
- net at D3.1 (K): now also Q5.3 (D); no longer Q5.1 (D)
- net at R1.1, R2.2: now also Q1.1 (G); no longer Q1.2 (G)
- net at D1.1 (K): now also Q1.3 (D); no longer Q1.1 (D)
- net HCMS_Reset: no longer names the net of U4.12 (*RESET)
- net HCMS_Reset: now also R28.1
- new net: Q13.1 (G), R29.2, R30.1
- new net: Q15.1 (G), R32.2, R33.1
- new net: D10.2 (A), D8.2 (A), D9.2 (A), R31.2
- new net: D11.2 (A), D12.2 (A), D13.2 (A), R34.2
- new net: D11.1 (K), D12.1 (K), D13.1 (K), Q15.3 (D)
- new net: D10.1 (K), D8.1 (K), D9.1 (K), Q13.3 (D)
- no-connect marks 25 -> 23

Commit message: Lot of Manual Routing
Connections:
- net +3V3: now also C3.1, C4.1, C7.1, C8.1, J1.4 (Pin_4), J2.4 (Pin_4), J3.4 (Pin_4), J4.4 (Pin_4), J5.1 (Pin_1), U2.20 (VCC), U5.20 (VCC)
- net +5V: no longer C3.1, C4.1, C7.1, C8.1, J1.4 (Pin_4), J2.4 (Pin_4), J3.4 (Pin_4), J4.4 (Pin_4), J5.1 (Pin_1), U2.20 (VCC), U5.20 (VCC)
- net Motor_LF_OutA: now also U1.42 (31_CTX3); no longer U1.41 (30_CRX3)
- net Motor_LF_OutB: now also U1.41 (30_CRX3); no longer U1.42 (31_CTX3)
- net Motor_LR_OutA: now also U1.44 (33_MCLK2); no longer U1.43 (32_OUT1B)
- net Motor_LR_OutB: now also U1.43 (32_OUT1B); no longer U1.44 (33_MCLK2)
- net Motor_RR_OutA: now also U1.40 (29_TX7); no longer U1.39 (28_RX7)
- net Motor_RR_OutB: now also U1.39 (28_RX7); no longer U1.40 (29_TX7)

Commit message: V2 Ready
Add new gyro board, remove motor stby. add LED Reset
Parts:
- removed C11, C13, C15, C17, C19, C5: 4.7uF, Capacitor_SMD:C_1206_3216Metric_Pad1.33x1.80mm_HandSolder, symbol Device:C_Small
- removed C12, C14, C16, C18, C20, C6: 0.1uF, Capacitor_SMD:C_1206_3216Metric_Pad1.33x1.80mm_HandSolder, symbol Device:C_Small
- removed D1, D13, D2, D3, D4, D5, D6, D8: IR, LED_THT:LED_D5.0mm_Horizontal_O3.81mm_Z9.0mm, symbol Device:LED
- removed J5: Conn_01x08_Pin, Connector_PinSocket_2.54mm:PinSocket_1x08_P2.54mm_Vertical, symbol Connector:Conn_01x08_Pin
- removed Q1, Q11, Q3, Q5, Q7, Q9: NMOS, Package_TO_SOT_SMD:SOT-23, symbol Simulation_SPICE:NMOS
- removed Q12, Q2: SFH300, LED_THT:LED_D5.0mm_Horizontal_O1.27mm_Z3.0mm_IRGrey, symbol Sensor_Optical:SFH300
- removed R1, R10, R14, R18, R22, R6: 47K, Resistor_SMD:R_1206_3216Metric_Pad1.30x1.75mm_HandSolder, symbol Device:R
- removed R11, R15, R19, R23, R3, R7: 51, Resistor_SMD:R_1206_3216Metric_Pad1.30x1.75mm_HandSolder, symbol Device:R
- removed R13, R17, R2, R21, R5, R9: 100, Resistor_SMD:R_1206_3216Metric_Pad1.30x1.75mm_HandSolder, symbol Device:R
- removed R24, R4: 1.8K, Resistor_SMD:R_1206_3216Metric_Pad1.30x1.75mm_HandSolder, symbol Device:R
- removed R28: 10K, Resistor_SMD:R_1206_3216Metric_Pad1.30x1.75mm_HandSolder, symbol Device:R
- added J6: Conn_01x10_Pin, Connector_PinHeader_2.54mm:PinHeader_1x10_P2.54mm_Vertical, symbol Connector:Conn_01x10_Pin
Connections:
- net IR_Reciever_Left_90 is gone; now on net Interface_Button1: U1.25 (18_A4_SDA0)
- net IR_Reciever_Right_90 is gone; now on net Interface_Button2: U1.30 (23_A9_CRX1_MCLK1)
- net +3V3: now also J6.1 (Pin_1)
- net GND: now also J6.2 (Pin_2)
- net Gyro_SCL: now also J6.3 (Pin_3)
- net Gyro_SDA: now also J6.4 (Pin_4)
- net Interface_Button1: no longer U1.45 (34_DAT1_MISO2)
- net Interface_Button2: no longer U1.46 (35_DAT0_MOSI2)
- net HCMS_RST: now reaches U4.12 (*RESET)
- net HCMS_RST: now also U1.10 (8_TX2_IN1)
- removed net Motor_STBY: U1.10 (8_TX2_IN1), U2.19 (STBY), U5.19 (STBY)
- no-connect marks 23 -> 29
Other:
- note added: "AD0"
- note added: "ECL"
- note added: "EDA"
- note added: "FSYNC"
- note added: "Gyroscope Module (GY-9250)"
- note added: "INT"
- note added: "VCC"
- note removed: "3V3"
- note removed: "CSB"
- note removed: "Gyroscope Module (GY-91)"
- note removed: "IR Emitter Circuit"
- note removed: "SDD/SAO"
- note removed: "VIN"
- moved on the sheet: C21, C22, C23, C24, D10, D11, D12, D9, Q10, Q13, Q15, Q4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
