File: Gmouse/Gmouse.kicad_sch (KiCad schematic)
At the start: 54 parts, among them J1 Motor_RF, J2 Motor_RR, J3 Motor_LF, J4 Motor_LR, J6 Conn_01x10_Pin, Q10 SFH300, Q13 NMOS, Q14 BC847, Q15 NMOS, Q4 SFH300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

Commit message: Most up-to-date Mouse Schematic and Layout
Parts:
- added R1, R2: 10k, symbol Device:R
Connections:
- net +3V3: now also R1.1, R2.1
- net at U5.19 (STBY): now also R2.2
- net at U2.19 (STBY): now also R1.2
- no-connect marks 29 -> 27
