File: Gmouse/Gmouse.kicad_pcb (KiCad board)
At the start: 4 copper layers, 80 x 100 mm, 61 parts, among them J1 Motor_RF, J2 Motor_RR, J3 Motor_LF, J4 Motor_LR, J5 Conn_01x08_Pin, Q10 SFH300, Q12 SFH300, Q13 NMOS, Q14 BC847, Q15 NMOS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

Commit message: Manufacturing Files for V1
Parts:
- added G***: LOGO, LOGO, B.Cu at (94.0, 104.0)
Other:
- board text added: "Pitt Robotics And Automation Society Aragya Goyal Olivia Sobek Ean Smith 40°26′39″N 79°57′11″W﻿"
- board text added: "{dblquote}Ka-Chow{dblquote}"

Commit message: V2 Ready
Add new gyro board, remove motor stby. add LED Reset
Parts:
- removed D13, D8: IR, LED_THT:LED_D5.0mm_Horizontal_O3.81mm_Z9.0mm
- removed J5: Conn_01x08_Pin, Connector_PinSocket_2.54mm:PinSocket_1x08_P2.54mm_Vertical
- removed Q12, Q2: SFH300, LED_THT:LED_D5.0mm_Horizontal_O1.27mm_Z3.0mm_IRGrey
- removed R24, R4: 1.8K, Resistor_SMD:R_1206_3216Metric_Pad1.30x1.75mm_HandSolder
- removed R28: 10K, Resistor_SMD:R_1206_3216Metric_Pad1.30x1.75mm_HandSolder
- added J6: Conn_01x10_Pin, Connector_PinHeader_2.54mm:PinHeader_1x10_P2.54mm_Vertical, F.Cu at (82.6, 53.9)
- moved R16 5.84 mm to (109.6, 52.0), turned to 90 degrees
- moved G*** 1.61 mm to (95.4, 103.2), turned to -90 degrees
Connections:
- U1 pad 10: Motor_STBY -> HCMS_RST
- U1 pad 25: IR_Reciever_Left_90 -> Interface_Button1
- U1 pad 30: IR_Reciever_Right_90 -> Interface_Button2
- U1 pad 45: Interface_Button1 -> unconnected-(U1-34_DAT1_MISO2-Pad45)
- U1 pad 46: Interface_Button2 -> unconnected-(U1-35_DAT0_MOSI2-Pad46)
- U2 pad 19: Motor_STBY -> unconnected-(U2-STBY-Pad19)
- U4 pad 12: Net-(U4-*RESET) -> HCMS_RST
- U5 pad 19: Motor_STBY -> unconnected-(U5-STBY-Pad19)
Routing:
- net HCMS_RST: track 0.00 -> 75.7 mm
- net Motor_STBY: track 74.9 -> 0.00 mm, vias 3 -> 0
- net IR_Reciever_Left_90: track 71.5 -> 0.00 mm, vias 1 -> 0
- net IR_Reciever_Right_90: track 28.9 -> 0.00 mm, vias 1 -> 0
- net +3V3: track 104.4 -> 76.9 mm, vias 18 -> 10
- net GND: track 132.0 -> 104.6 mm, vias 32 -> 25
- net Motor_LR_PWM: track 84.6 -> 62.4 mm
- net Interface_Button2: track 72.8 -> 61.3 mm
- net Net-(D11-A): track 31.3 -> 21.8 mm
- net Net-(D10-K): track 31.3 -> 23.0 mm
- net Gyro_SDA: track 32.1 -> 38.6 mm, vias 0 -> 1
- net Gyro_SCL: track 34.9 -> 41.4 mm, vias 0 -> 1
- net Net-(D10-A): track 26.7 -> 20.3 mm
- net Net-(D11-K): track 32.9 -> 27.7 mm, vias 0 -> 1
- net Interface_Button1: track 60.0 -> 55.6 mm, vias 0 -> 1
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